Commit message: 修改urdf中的Continuous为Revolute

File: fanuc_m20id35_support/urdf/fanuc_m20id35_klampt.urdf (robot description, URDF)
Before this commit: robot fanuc_m20id35_support, 9 links, 8 joints
Joints:
- joint joint_1: type continuous -> revolute
- joint joint_2: type continuous -> revolute
- joint joint_3: type continuous -> revolute
- joint joint_4: type continuous -> revolute
- joint joint_5: type continuous -> revolute
- joint joint_6: type continuous -> revolute
